File: ESP32-Simple-Thermostat-PCB/ESP32-Simple-Thermostat-PCB.kicad_pcb (KiCad board)
At the start: 2 copper layers, 133 x 89.5 mm, 48 parts, among them J1 External Relays, J2 Screw_Terminal_9_P3.50mm, J3 DS18B20, J4 3.2 lcd tft, K1 G5Q-1A, K2 G5Q-1A, K3 G5Q-1A, K4 G5Q-1A, K5 G5Q-1A, K6 G5Q-1A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

Commit message: Standardize project naming to ESP32 Simple Thermostat
- Updated display text, serial messages, and MQTT device model
- Updated all web interface page titles and headers
- Consistent branding across documentation and code
Parts:
- J1: value External Relays -> PINHD_1x18_Male
Connections:
- A1 pad 21: unconnected-(A1-ADC1_CH4/D32-Pad21) -> D32
- A1 pad 22: D32 -> D33
- J4 pad 8: +5V -> D32
- R6 pad 2: D32 -> D33
Routing:
- net D33: track 0.00 -> 68.0 mm, vias 0 -> 1
- net D32: track 68.0 -> 41.9 mm, vias 1 -> 0
- net +5V: track 360.0 -> 343.8 mm
Changed lines of the file:
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@@
 	(net 1 "unconnected-(A1-RX2{slash}GPIO16-Pad6)")
 	(net 2 "CS_15")
-	(net 3 "unconnected-(A1-ADC1_CH4{slash}D32-Pad21)")
+	(net 3 "D33")
 	(net 4 "D32")
 	(net 5 "GND")
@@
 			)
 		)
-		(property "Value" "External Relays"
+		(property "Value" "PINHD_1x18_Male"
 			(at 0 45.56 0)
 			(layer "F.Fab")
@@
 			(layers "*.Cu" "*.Mask")
 			(remove_unused_layers no)
-			(net 3 "unconnected-(A1-ADC1_CH4{slash}D32-Pad21)")
+			(net 4 "D32")
 			(pinfunction "ADC1_CH4/D32")
 			(pintype "bidirectional")
@@
 			(layers "*.Cu" "*.Mask")
 			(remove_unused_layers no)
-			(net 4 "D32")
-			(pinfunction "ADC1_CH4/D32")
+			(net 3 "D33")
+			(pinfunction "ADC1_CH4/D33")
 			(pintype "bidirectional")
 		)
@@
 			(layers "*.Cu" "*.Mask")
 			(remove_unused_layers no)
-			(net 4 "D32")
+			(net 3 "D33")
 			(pintype "passive")
 		)
@@
 			(layers "*.Cu" "*.Mask")
 			(remove_unused_layers no)
-			(net 8 "+5V")
+			(net 4 "D32")
 			(pintype "passive")
 		)
@@
 		(width 0.2)
 		(layer "F.Cu")
-		(net 4)
+		(net 3)
 	)
 	(segment
@@
 		(width 0.2)
 		(layer "F.Cu")
-		(net 4)
+		(net 3)
 	)
 	(segment
@@
 		(width 0.2)
 		(layer "F.Cu")
-		(net 4)
+		(net 3)
 	)
 	(segment
@@
 		(width 0.2)
 		(layer "F.Cu")
-		(net 4)
+		(net 3)
 	)
 	(segment
@@
 		(width 0.2)
 		(layer "F.Cu")
-		(net 4)
+		(net 3)
 	)
 	(segment
@@
 		(width 0.2)
 		(layer "F.Cu")
-		(net 4)
+		(net 3)
 	)
 	(segment
@@
 		(width 0.2)
 		(layer "F.Cu")
-		(net 4)
+		(net 3)
 	)
 	(via
@@
 		(drill 0.3)
 		(layers "F.Cu" "B.Cu")
-		(net 4)
+		(net 3)
 	)
 	(segment
@@
 		(width 0.2)
 		(layer "B.Cu")
-		(net 4)
+		(net 3)
 	)
 	(segment
@@
 		(width 0.2)
 		(layer "B.Cu")
-		(net 4)
+		(net 3)
 	)
 	(segment
@@
 		(width 0.2)
 		(layer "B.Cu")
-		(net 4)
+		(net 3)
 	)
 	(segment
@@
 		(width 0.2)
 		(layer "B.Cu")
+		(net 3)
+	)
+	(segment
+		(start 105.8506 62.385)
+		(end 98.47276 62.385)
+		(width 0.2)
+		(layer "F.Cu")
+		(net 4)
+	)
+	(segment
+		(start 98.47276 62.385)
+		(end 96.28676 64.571)
+		(width 0.2)
+		(layer "F.Cu")
+		(net 4)
+	)
+	(segment
+		(start 67.901 65.359)
+		(end 66 67.26)
+		(width 0.2)
+		(layer "F.Cu")
+		(net 4)
+	)
+	(segment
+		(start 96.28676 64.571)
+		(end 89.929 64.571)
+		(width 0.2)
+		(layer "F.Cu")
+		(net 4)
+	)
+	(segment
+		(start 89.929 64.571)
+		(end 89.141 65.359)
+		(width 0.2)
+		(layer "F.Cu")
+		(net 4)
+	)
+	(segment
+		(start 89.141 65.359)
+		(end 67.901 65.359)
+		(width 0.2)
+		(layer "F.Cu")
 		(net 4)
 	)
@@
 	)
 	(segment
-		(start 81.55 65.8133)
-		(end 67.4467 65.8133)
-		(width 0.2)
-		(layer "F.Cu")
-		(net 8)
-	)
-	(segment
 		(start 81.5 88)
 		(end 81.5 86)
@@
 		(layer "F.Cu")
 		(net 8)
-	)
-	(segment
-		(start 67.4467 65.8133)
-		(end 66 67.26)
-		(width 0.2)
-		(layer "F.Cu")
-		(net 8)
